Commit message: Changes for using namespaces and collision detection

File: urdf/ur10e.urdf (robot description, URDF)
Before this commit: robot ur10e, 13 links, 12 joints
Links:
- link base_link_inertia: geometry collision mesh filename=package://ur_description/meshes/ur10e/collision/base.stl scale=1.2 1.2 1.2; visual mesh filename=package://ur_description/meshes/ur10e/visual/base.dae
- link forearm_link: geometry collision mesh filename=package://ur_description/meshes/ur10e/collision/forearm.stl scale=1.2 1.2 1.2; visual mesh filename=package://ur_description/meshes/ur10e/visual/forearm.dae
- link shoulder_link: geometry collision mesh filename=package://ur_description/meshes/ur10e/collision/shoulder.stl scale=1.2 1.2 1.2; visual mesh filename=package://ur_description/meshes/ur10e/visual/shoulder.dae
- link upper_arm_link: geometry collision mesh filename=package://ur_description/meshes/ur10e/collision/upperarm.stl scale=1.2 1.2 1.2; visual mesh filename=package://ur_description/meshes/ur10e/visual/upperarm.dae
- link wrist_1_link: geometry collision mesh filename=package://ur_description/meshes/ur10e/collision/wrist1.stl scale=1.2 1.2 1.2; visual mesh filename=package://ur_description/meshes/ur10e/visual/wrist1.dae
- link wrist_2_link: geometry collision mesh filename=package://ur_description/meshes/ur10e/collision/wrist2.stl scale=1.2 1.2 1.2; visual mesh filename=package://ur_description/meshes/ur10e/visual/wrist2.dae
- link wrist_3_link: geometry collision mesh filename=package://ur_description/meshes/ur10e/collision/wrist3.stl scale=1.2 1.2 1.2; visual mesh filename=package://ur_description/meshes/ur10e/visual/wrist3.dae
