Commit message: bim model

File: urdf/BIM_model.urdf (robot description, URDF)
Before this commit: robot BIM_model, 1 links, 0 joints
Links:
- removed link base_link
- added link bim; collision mesh filename=package://ur_arm_control/urdf/example_building.stl; visual mesh filename=package://ur_arm_control/urdf/example_building.stl
